File: PCB Design/Balance_Bot/Balance_Bot.kicad_sch (KiCad schematic)
At the start: 2 parts, among them U1 MPU-6050

Commit message: Code and KiCad
Parts:
- removed ESP1: ~, ME507A:ESP32_NodeMCU_KeeYees, symbol ME507A:ESP32_Node_KY
- added A1: Adafruit_Feather_HUZZAH32_ESP32, Module:Adafruit_Feather, symbol MCU_Module:Adafruit_Feather_HUZZAH32_ESP32
- added C1: 2.2 nF, Capacitor_SMD:C_0805_2012Metric, symbol Device:C
- added C2: 0.1uF, Capacitor_SMD:C_0805_2012Metric, symbol Device:C
- added C3, C4: 10 uF, Capacitor_SMD:C_0805_2012Metric, symbol Device:C
- added C5: 0.1 uF, Capacitor_SMD:C_0805_2012Metric, symbol Device:C
- added C6: 47uF/63V, symbol Device:C_Polarized
- added C7: 0.1uF/50V, Capacitor_SMD:C_0805_2012Metric, symbol Device:C
- added D1: GREEN, LED_SMD:LED_0805_2012Metric, symbol Device:LED
- added J1: DC Motor A, symbol Connector:Screw_Terminal_01x02
- added J2: DC Motor B, symbol Connector:Screw_Terminal_01x02
- added J3: Motor Power, symbol Connector:Screw_Terminal_01x02
- added JP1: Open, Jumper:SolderJumper-2_P1.3mm_Open_RoundedPad1.0x1.5mm, symbol Jumper:SolderJumper_2_Open
- added JP2, JP3: Bridged, Jumper:SolderJumper-2_P1.3mm_Bridged_RoundedPad1.0x1.5mm, symbol Jumper:SolderJumper_2_Bridged
- added Q1, Q2: BSS138, Package_TO_SOT_SMD:SOT-23, symbol Transistor_FET:BSS138
- added R1, R2, R3, R4, R5, R6: 10k, Resistor_SMD:R_0805_2012Metric, symbol Device:R
- added R7, R8: 30K, Resistor_SMD:R_0805_2012Metric, symbol Device:R
- added U2: AP2112K-3.3, Package_TO_SOT_SMD:SOT-23-5, symbol Regulator_Linear:AP2112K-3.3
- added U3, U4: DRV8871DDA, Package_SO:Texas_HTSOP-8-1EP_3.9x4.9mm_P1.27mm_EP2.95x4.9mm_Mask2.4x3.1mm_ThermalVias, symbol Driver_Motor:DRV8871DDA
Connections:
- net 3V3 is gone; now on net +3.3V: U1.13 (VDD)
- net GND: now also A1.4 (GND), C1.1, C2.1, C3.2, C4.2, C5.2, C6.2, C7.1, D1.1 (K), J3.2 (Pin_2), JP2.2 (B), JP3.2 (B), R1.2, R7.2, R8.2, U2.2 (GND), U3.1 (GND), U3.7 (GND), U3.9 (GND), U4.1 (GND), U4.7 (GND), U4.9 (GND)
- net SDA_3V: now reaches U1.24 (SDA)
- net SDA_3V: now also Q1.2 (S), R6.2
- net SCL_3V: now reaches U1.23 (SCL)
- net SCL_3V: now also Q2.2 (S), R5.2
- net CLKIN: now reaches U1.1 (CLKIN)
- net CLKIN: now also JP3.1 (A)
- net at U1.10 (REGOUT): now also C2.2
- net FSYNC: now reaches U1.11 (FSYNC)
- net FSYNC: now also JP2.1 (A)
- net INT: now reaches U1.12 (INT)
- net at U1.20 (CPOUT): now also C1.2
- net SDA_EXIT: now reaches U1.6 (AUX_DA)
- net SCL_EXT: now reaches U1.7 (AUX_CL)
- net +3.3V: now reaches U1.8 (VLOGIC)
- net +3.3V: now also C4.1, C5.1, JP1.2 (B), Q1.1 (G), Q2.1 (G), R2.1, R5.1, R6.1, U2.5 (VOUT)
- net AD0: now reaches U1.9 (AD0)
- net AD0: now also JP1.1 (A), R1.1
- new net: J2.1 (Pin_1), U4.6 (OUT1)
- new net: J2.2 (Pin_2), U4.8 (OUT2)
- new net: R7.1, U3.4 (ILIM)
- new net: J1.1 (Pin_1), U3.6 (OUT1)
- new net: J1.2 (Pin_2), U3.8 (OUT2)
- new net: R8.1, U4.4 (ILIM)
- new net: D1.2 (A), R2.2
- new net IN1_A: U3.3 (IN1), U4.3 (IN1)
- new net IN2_A: U3.2 (IN2), U4.2 (IN2)
- new net MOTOR_POWER: C6.1, C7.2, J3.1 (Pin_1), U3.5 (VM), U4.5 (VM)
- new net SCL: A1.18 (SCL/IO22), Q2.3 (D), R3.2
- new net SDA: A1.17 (SDA/IO23), Q1.3 (D), R4.2
- new net VCC: C3.1, R3.1, R4.1, U2.1 (VIN), U2.3 (EN)
Other:
- note added: "2X C7 CLOSE TO EACH DRIVER"
- note added: "I2C ADDRESS"
- note added: "I2C PULLUPS & SHIFT"
- note added: "MOTOR DRIVER"
- note added: "MPU-6050"
- note added: "ON LED"
- note added: "POWER SUPPLY"
- company: ME 507 -> Vormbaum & Raventos - ME 507
- moved on the sheet: U1
