File: PCB_Design/Balance_Bot/Balance_Bot.kicad_pcb (KiCad board)
At the start: 2 copper layers, 20 parts, among them Q1 BSS138, Q2 BSS138, U1 MPU-6050, U2 AP2112K-3.3

Commit message: board stuff
Parts:
- removed JP1: Open, Jumper:SolderJumper-2_P1.3mm_Open_RoundedPad1.0x1.5mm
- removed JP2, JP3: Bridged, Jumper:SolderJumper-2_P1.3mm_Bridged_RoundedPad1.0x1.5mm
- removed Q1, Q2: BSS138, Package_TO_SOT_SMD:SOT-23
- removed R3, R4, R5, R6: 10k, Resistor_SMD:R_0805_2012Metric
- added C6: 0.1uF/12V, Capacitor_SMD:C_0805_2012Metric, F.Cu at (181.6, 100.8)
- added C7: 47uF/12V, Capacitor_SMD:CP_Elec_5x5.3, F.Cu at (175.6, 85.6)
- added C9: 47uF/12V, Capacitor_SMD:CP_Elec_5x5.3, F.Cu at (176.4, 113.2)
- added J1: LEFT_MOTOR, TerminalBlock_Phoenix:TerminalBlock_Phoenix_MPT-0,5-6-2.54_1x06_P2.54mm_Horizontal, F.Cu at (190.5, 83.1)
- added J2: RIGHT_MOTOR, TerminalBlock_Phoenix:TerminalBlock_Phoenix_MPT-0,5-6-2.54_1x06_P2.54mm_Horizontal, F.Cu at (190.5, 115.1)
- added J3: 12V_BAT, TerminalBlock_Phoenix:TerminalBlock_Phoenix_MPT-0,5-2-2.54_1x02_P2.54mm_Horizontal, F.Cu at (190.0, 93.7)
- added J4: Conn_01x08_Socket, Connector_PinSocket_1.00mm:PinSocket_1x08_P1.00mm_Vertical, F.Cu at (158.8, 132.1)
- added R10: 10k, Resistor_SMD:R_0805_2012Metric, F.Cu at (174.5, 132.6)
- added R11: 10k, Resistor_SMD:R_0805_2012Metric, F.Cu at (176.5, 138.4)
- added R8: 30K, Resistor_SMD:R_0805_2012Metric, F.Cu at (169.7, 129.1)
- added U4: DRV8871DDA, Package_SO:Texas_HTSOP-8-1EP_3.9x4.9mm_P1.27mm_EP2.95x4.9mm_Mask2.4x3.1mm_ThermalVias, F.Cu at (170.8, 103.6)
- C4: value 10 uF -> 0.1 uF
- C5: value 0.1 uF -> 0.1uF/12V
- R1: value 10k -> 30K
- U2: value AP2112K-3.3 -> DRV8871DDA; footprint Package_TO_SOT_SMD:SOT-23-5 -> Package_SO:Texas_HTSOP-8-1EP_3.9x4.9mm_P1.27mm_EP2.95x4.9mm_Mask2.4x3.1mm_ThermalVias
- moved D1 60.2 mm to (160.8, 112.8)
- moved C1 58.4 mm to (186.4, 135.6), turned to 180 degrees
- moved C2 55.5 mm to (186.4, 140.2), turned to 180 degrees
- moved C3 52.9 mm to (165.3, 129.2)
- moved A1 52.0 mm to (150.6, 129.3), turned to 180 degrees
- moved C4 44.9 mm to (167.6, 137.2)
- moved R1 43.6 mm to (175.8, 121.4)
- moved U1 42.5 mm to (182.9, 126.9)
- moved C5 39.6 mm to (180.6, 78.7)
- moved R2 31.4 mm to (169.7, 126.1)
- moved U2 4.55 mm to (170.1, 76.2)
Connections:
- A1 pad 10: unconnected-(A1-IO4/A5-Pad10) -> OUT_B_LEFT
- A1 pad 17: unconnected-(A1-SDA/IO23-Pad17) -> SDA
- A1 pad 18: unconnected-(A1-SCL/IO22-Pad18) -> SCL
- A1 pad 19: unconnected-(A1-A6/IO14-Pad19) -> IN1_RIGHT
- A1 pad 2: unconnected-(A1-3V3-Pad2) -> +3.3V
- A1 pad 20: unconnected-(A1-A7/IO32-Pad20) -> IN2_RIGHT
- A1 pad 21: unconnected-(A1-A8/IO15-Pad21) -> IN1_LEFT
- A1 pad 22: unconnected-(A1-A9/IO33-Pad22) -> IN2_LEFT
- A1 pad 7: unconnected-(A1-I34/A2-Pad7) -> OUT_A_RIGHT
- A1 pad 8: unconnected-(A1-I39/A3-Pad8) -> OUT_B_RIGHT
- A1 pad 9: unconnected-(A1-IO36/A4-Pad9) -> OUT_A_LEFT
- C3 pad 1: VCC -> +3.3V
- C5 pad 1: +3.3V -> 12V_BAT
- R1 pad 1: AD0 -> Net-(U2-ILIM)
- U1 pad 1: CLKIN -> GND
- U1 pad 11: FSYNC -> GND
- U1 pad 23: SCL_3V -> SCL
- U1 pad 24: SDA_3V -> SDA
- U1 pad 6: SDA_EXIT -> GND
- U1 pad 7: SCL_EXT -> GND
- U1 pad 9: AD0 -> GND
- U2 pad 1: VCC -> GND
- U2 pad 2: GND -> IN2_LEFT
- U2 pad 3: VCC -> IN1_LEFT
- U2 pad 4: unconnected-(U2-NC-Pad4) -> Net-(U2-ILIM)
- U2 pad 5: +3.3V -> 12V_BAT

Commit message: board design
Parts:
- moved R1 46.3 mm to (160.8, 77.7), turned to 180 degrees
- moved R2 41.1 mm to (164.9, 85.3), turned to 180 degrees
- moved R8 32.6 mm to (160.4, 97.8), turned to 180 degrees
- moved J4 31.5 mm to (190.0, 127.7), turned to 180 degrees
- moved D1 27.5 mm to (159.6, 85.3)
- moved R11 21.5 mm to (165.6, 119.9), turned to -90 degrees
- moved C1 21.4 mm to (172.0, 119.9), turned to -90 degrees
- moved C2 16.3 mm to (170.9, 135.1), turned to 90 degrees
- moved U1 12.3 mm to (170.7, 128.0)
- moved R10 11.7 mm to (178.7, 121.7), turned to 180 degrees
- moved C4 10.0 mm to (158.0, 134.4), turned to -90 degrees
- moved U4 7.81 mm to (170.8, 95.8)
- moved C9 6.54 mm to (176.4, 106.7)
- moved J2 6.10 mm to (190.5, 109.0)
- moved C3 5.71 mm to (162.8, 134.4), turned to -90 degrees
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Connections:
- J4 pad 1: +3V3 -> +3.3V
Routing:
- net +3.3V: track 0.00 -> 164.2 mm
- net SDA: track 0.00 -> 161.3 mm
- net SCL: track 0.00 -> 106.8 mm
- net GND: track 0.00 -> 64.9 mm, vias 0 -> 8
- net Net-(U1-CPOUT): track 0.00 -> 5.44 mm
- net Net-(U1-REGOUT): track 0.00 -> 4.21 mm
- added copper zone on B.Cu, net GND
Other:
- board outline added: 116.3 x 98.3 mm

Commit message: board
Parts:
- added H1: MountingHole, MountingHole:MountingHole_3.2mm_M3, F.Cu at (127.8, 65.8)
- added H2: MountingHole, MountingHole:MountingHole_3.2mm_M3, F.Cu at (200.4, 65.5)
- added H3: MountingHole, MountingHole:MountingHole_3.2mm_M3, F.Cu at (199.6, 141.5)
- added H4: MountingHole, MountingHole:MountingHole_3.2mm_M3, F.Cu at (128.0, 141.5)
- C5, C6: value 0.1uF/12V -> 0.1uF/16V
- C7, C9: value 47uF/12V -> 47uF/16V; footprint Capacitor_SMD:CP_Elec_5x5.3 -> Capacitor_THT:CP_Radial_D6.3mm_P2.50mm
- J4: footprint Connector_PinSocket_1.00mm:PinSocket_1x08_P1.00mm_Vertical -> Connector_PinSocket_2.54mm:PinSocket_1x08_P2.54mm_Vertical
- moved C6 17.4 mm to (164.1, 103.1), turned to 180 degrees
- moved C5 17.0 mm to (164.3, 78.5), turned to 180 degrees
- moved U4 10.2 mm to (160.9, 98.1)
- moved U2 9.91 mm to (161.1, 73.4)
- moved C7 9.82 mm to (169.3, 78.2)
- moved J4 9.44 mm to (190.8, 137.2)
- moved C9 7.99 mm to (169.2, 103.1)
- moved R8 6.41 mm to (156.5, 102.9), turned to -90 degrees
- moved R1 4.06 mm to (156.7, 78.1), turned to -90 degrees
- moved D1 1.91 mm to (157.7, 85.9), turned to -90 degrees
- moved R2 1.46 mm to (163.6, 85.9), turned to 90 degrees
- moved J1 1.27 mm to (190.5, 84.6)
- moved J3 0.51 mm to (190.5, 91.7)
Routing:
- net +3.3V: track 164.2 -> 292.1 mm, vias 0 -> 1
- net OUT_A_LEFT: track 0.00 -> 101.2 mm
- net OUT_B_LEFT: track 0.00 -> 97.0 mm, vias 0 -> 1
- net OUT_B_RIGHT: track 0.00 -> 78.4 mm, vias 0 -> 1
- net OUT_A_RIGHT: track 0.00 -> 66.4 mm, vias 0 -> 1
- net IN2_LEFT: track 0.00 -> 61.4 mm
- net 12V_BAT: track 0.00 -> 60.0 mm, vias 0 -> 4
- net IN1_LEFT: track 0.00 -> 56.3 mm
- net IN2_RIGHT: track 0.00 -> 47.1 mm
- net IN1_RIGHT: track 0.00 -> 33.2 mm, vias 0 -> 2
- net Net-(J2-Pin_2): track 0.00 -> 31.5 mm
- net Net-(J1-Pin_2): track 0.00 -> 31.5 mm
- net Net-(J2-Pin_1): track 0.00 -> 30.0 mm
- net Net-(J1-Pin_1): track 0.00 -> 30.0 mm
- net Net-(D1-A): track 0.00 -> 14.2 mm
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- added copper zone on F.Cu, net 12V_BAT
- added copper zone on F.Cu, net GND
- added copper zone on F.Cu, net Net-(J1-Pin_1)
- added copper zone on F.Cu, net Net-(J1-Pin_2)
- added copper zone on F.Cu, net Net-(J2-Pin_1)
- added copper zone on F.Cu, net Net-(J2-Pin_2)
Other:
- board size 116.3 x 98.3 mm -> 81.5 x 85.1 mm
- board text added: "+ -"
- board text added: "M1 M2 Vcc A B GND"
