File: PCB_Design/Balance_Bot/Balance_Bot.kicad_pcb (KiCad board)
At the start: 2 copper layers, 81.5 x 85.1 mm, 26 parts, among them J1 LEFT_MOTOR, J2 RIGHT_MOTOR, J3 12V_BAT, J4 Conn_01x08_Socket, U1 MPU-6050, U2 DRV8871DDA, U4 DRV8871DDA

Commit message: PCB update
Thickened some power traces to 24mil

Added white dot next to GND pins on motor drivers to tell us orientation

Added square showing MPU breakout orientation
Other:
- board text added: "MPU6050 Breakout"
Changed lines of the file:
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@@
     )
   )
+  (gr_circle (center 155.936532 96.212233) (end 156.317532 96.212233)
+    (stroke (width 0.15) (type solid)) (fill solid) (layer "F.SilkS"))
+  (gr_rect (start 176.244723 117.451492) (end 192.864092 139.264414)
+    (stroke (width 0.15) (type default)) (fill none) (layer "F.SilkS"))
+  (gr_circle (center 156.132593 71.51846) (end 156.513593 71.51846)
+    (stroke (width 0.15) (type solid)) (fill solid) (layer "F.SilkS"))
   (gr_rect (start 123.317 60.96) (end 204.851 146.05)
     (stroke (width 0.1) (type default)) (fill none) (layer "Edge.Cuts"))
+  (gr_text "MPU6050 Breakout" (at 177.846068 116.672458) (layer "F.SilkS")
+    (effects (font (size 1 1) (thickness 0.15)) (justify left bottom))
+  )
   (gr_text "M1 M2 Vcc A B GND" (at 196.088 85.852 90) (layer "F.SilkS")
     (effects (font (size 1 1) (thickness 0.15)) (justify left bottom))
@@
   (segment (start 170.938 129.966) (end 170.938 134.174) (width 0.25) (layer "F.Cu") (net 41))
   (segment (start 175.768 129.286) (end 172.658 129.286) (width 0.25) (layer "F.Cu") (net 42))
-  (segment (start 157.988 130.81) (end 161.163 127.635) (width 0.25) (layer "F.Cu") (net 42))
-  (segment (start 166.878 132.334) (end 169.926 132.334) (width 0.25) (layer "F.Cu") (net 42))
+  (segment (start 157.988 130.81) (end 161.163 127.635) (width 0.6096) (layer "F.Cu") (net 42))
+  (segment (start 166.878 132.334) (end 169.926 132.334) (width 0.254) (layer "F.Cu") (net 42))
   (segment (start 196.85 80.518) (end 193.548 80.518) (width 0.25) (layer "F.Cu") (net 42))
   (segment (start 162.814 131.064) (end 163.703 130.175) (width 0.61) (layer "F.Cu") (net 42))
@@
   (segment (start 160.274 117.094) (end 165.608 117.094) (width 0.61) (layer "F.Cu") (net 42))
   (segment (start 193.548 80.518) (end 192.532 79.502) (width 0.25) (layer "F.Cu") (net 42))
-  (segment (start 177.546 142.24) (end 177.546 137.16) (width 0.25) (layer "F.Cu") (net 42))
+  (segment (start 177.546 142.24) (end 177.546 137.16) (width 0.6096) (layer "F.Cu") (net 42))
   (segment (start 154.432 126.746) (end 154.432 142.24) (width 0.61) (layer "F.Cu") (net 42))
-  (segment (start 190.754 137.16) (end 177.546 137.16) (width 0.25) (layer "F.Cu") (net 42))
+  (segment (start 190.754 137.16) (end 177.546 137.16) (width 0.6096) (layer "F.Cu") (net 42))
   (segment (start 172.658 129.286) (end 172.638 129.266) (width 0.25) (layer "F.Cu") (net 42))
   (segment (start 160.274 126.746) (end 160.274 117.094) (width 0.61) (layer "F.Cu") (net 42))
@@
   (segment (start 153.416 89.916) (end 163.576 89.916) (width 0.25) (layer "F.Cu") (net 42))
   (segment (start 165.862 89.916) (end 168.656 92.71) (width 0.25) (layer "F.Cu") (net 42))
-  (segment (start 157.988 133.416) (end 157.988 130.81) (width 0.25) (layer "F.Cu") (net 42))
+  (segment (start 157.988 133.416) (end 157.988 130.81) (width 0.6096) (layer "F.Cu") (net 42))
   (segment (start 145.796 87.63) (end 151.13 87.63) (width 0.25) (layer "F.Cu") (net 42))
   (segment (start 169.926 132.334) (end 169.926 130.81) (width 0.25) (layer "F.Cu") (net 42))
@@
   (segment (start 169.926 130.81) (end 169.938 130.798) (width 0.25) (layer "F.Cu") (net 42))
   (segment (start 179.625 121.666) (end 181.864 121.666) (width 0.61) (layer "F.Cu") (net 42))
-  (segment (start 154.432 142.24) (end 177.546 142.24) (width 0.25) (layer "F.Cu") (net 42))
+  (segment (start 154.432 142.24) (end 177.546 142.24) (width 0.6096) (layer "F.Cu") (net 42))
   (via (at 145.796 87.63) (size 0.8) (drill 0.4) (layers "F.Cu" "B.Cu") (net 42))
   (segment (start 150.622 126.746) (end 145.796 126.746) (width 0.25) (layer "B.Cu") (net 42))

Commit message: Board stuff
Parts:
- removed C2: 0.1uF, Capacitor_SMD:C_0805_2012Metric
- removed C4: 0.1 uF, Capacitor_SMD:C_0805_2012Metric
- added 0.1 uF: 0.1uF, Capacitor_SMD:C_0805_2012Metric, F.Cu at (164.8, 123.1)
- added 0.1 uF: 0.1 uF, Capacitor_SMD:C_0805_2012Metric, F.Cu at (168.8, 118.9)
- moved R10 58.2 mm to (126.5, 96.0), turned to 0 degrees
- moved R11 49.8 mm to (126.5, 89.0), turned to 0 degrees
- moved U1 13.2 mm to (162.5, 117.6)
- moved C3 11.5 mm to (160.4, 123.1), turned to 180 degrees
- moved C1 10.7 mm to (164.2, 112.5), turned to 180 degrees
- moved J4 4.47 mm to (190.5, 132.7)
- moved R2 2.39 mm to (161.2, 85.6)
- moved D1 0.37 mm to (158.0, 85.6), turned to 90 degrees
- moved C9 0.17 mm to (169.3, 103.0)
Connections:
- A1 pad 23: unconnected-(A1-A10/IO27-Pad23) -> INT
- J4 pad 8: unconnected-(J4-Pin_8-Pad8) -> INT
Routing:
- net INT: track 0.00 -> 91.6 mm, vias 0 -> 1
- net SDA: track 162.2 -> 96.6 mm, vias 0 -> 1
- net +3.3V: track 292.1 -> 232.3 mm
- net GND: track 72.9 -> 17.4 mm, vias 59 -> 213
- net SCL: track 115.9 -> 92.8 mm, vias 0 -> 1
- net IN2_RIGHT: track 47.1 -> 28.6 mm, vias 0 -> 2
- net OUT_B_RIGHT: track 78.4 -> 67.1 mm, vias 1 -> 0
- net Net-(D1-A): track 14.2 -> 3.21 mm
- net IN2_LEFT: track 61.4 -> 69.7 mm, vias 0 -> 1
- net IN1_LEFT: track 56.3 -> 61.5 mm, vias 0 -> 1
- net IN1_RIGHT: track 33.2 -> 30.1 mm
- net Net-(U1-CPOUT): track 5.44 -> 3.18 mm
- net Net-(J2-Pin_2): track 31.5 -> 29.4 mm
- net Net-(J1-Pin_2): track 31.5 -> 29.6 mm
- net OUT_B_LEFT: track 97.0 -> 98.9 mm, vias 1 -> 0
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Other:
- board size 81.5 x 85.1 mm -> 85.3 x 85.1 mm

Commit message: final board
Parts:
- added H5: IMU MountingHole, MountingHole:MountingHole_3.2mm_M3, F.Cu at (178.6, 131.3)
- added H6: IMU MountingHole, MountingHole:MountingHole_3.2mm_M3, F.Cu at (178.6, 116.0)
- C2, C4: renamed from 0.1 uF
- moved H4 5.24 mm to (122.9, 142.7)
- moved H1 5.02 mm to (122.9, 64.4)
- moved H3 2.01 mm to (201.2, 142.7)
- moved H2 1.37 mm to (201.2, 64.4)
- moved J4 0.15 mm to (190.3, 132.7)
Routing:
- net SCL: track 92.8 -> 97.5 mm
- net SDA: track 96.6 -> 100.5 mm
- net +3.3V: track 232.3 -> 235.9 mm
- net GND: vias 213 -> 227
