File: PCB_Design/Balance_Bot/Balance_Bot.kicad_sch (KiCad schematic)
At the start: 29 parts, among them J1 DC Motor A, J2 DC Motor B, J3 Motor Power, Q1 BSS138, Q2 BSS138, U1 MPU-6050, U2 AP2112K-3.3, U3 DRV8871DDA, U4 DRV8871DDA

Commit message: board design
Parts:
- removed C6: 47uF/63V, symbol Device:C_Polarized
- removed C7: 0.1uF/50V, Capacitor_SMD:C_0805_2012Metric, symbol Device:C
- removed J1: DC Motor A, symbol Connector:Screw_Terminal_01x02
- removed J2: DC Motor B, symbol Connector:Screw_Terminal_01x02
- removed JP1: Open, Jumper:SolderJumper-2_P1.3mm_Open_RoundedPad1.0x1.5mm, symbol Jumper:SolderJumper_2_Open
- removed JP2, JP3: Bridged, Jumper:SolderJumper-2_P1.3mm_Bridged_RoundedPad1.0x1.5mm, symbol Jumper:SolderJumper_2_Bridged
- removed Q1, Q2: BSS138, Package_TO_SOT_SMD:SOT-23, symbol Transistor_FET:BSS138
- removed R3, R4, R5, R6: 10k, Resistor_SMD:R_0805_2012Metric, symbol Device:R
- removed R7: 30K, Resistor_SMD:R_0805_2012Metric, symbol Device:R
- removed U2: AP2112K-3.3, Package_TO_SOT_SMD:SOT-23-5, symbol Regulator_Linear:AP2112K-3.3
- removed U3: DRV8871DDA, Package_SO:Texas_HTSOP-8-1EP_3.9x4.9mm_P1.27mm_EP2.95x4.9mm_Mask2.4x3.1mm_ThermalVias, symbol Driver_Motor:DRV8871DDA
- added C6: 0.1uF/12V, Capacitor_SMD:C_0805_2012Metric, symbol Device:C
- added C7, C9: 47uF/12V, symbol Device:C_Polarized
- added H1, H2, H3, H4: MountingHole_Pad, symbol Mechanical:MountingHole_Pad
- added J1: LEFT_MOTOR, TerminalBlock_Phoenix:TerminalBlock_Phoenix_PT-1,5-6-3.5-H_1x06_P3.50mm_Horizontal, symbol Connector:Screw_Terminal_01x06
- added J2: RIGHT_MOTOR, TerminalBlock_Phoenix:TerminalBlock_Phoenix_PT-1,5-6-3.5-H_1x06_P3.50mm_Horizontal, symbol Connector:Screw_Terminal_01x06
- added R10, R11: 10k, Resistor_SMD:R_0805_2012Metric, symbol Device:R
- added U2: DRV8871DDA, Package_SO:Texas_HTSOP-8-1EP_3.9x4.9mm_P1.27mm_EP2.95x4.9mm_Mask2.4x3.1mm_ThermalVias, symbol Driver_Motor:DRV8871DDA
- C4: value 10 uF -> 0.1 uF
- C5: value 0.1 uF -> 0.1uF/12V
- J3: value Motor Power -> 12V_BAT
- R1: value 10k -> 30K
Connections:
- net CLKIN is gone; now on net GND: U1.1 (CLKIN)
- net FSYNC is gone; now on net GND: U1.11 (FSYNC)
- net IN1_A is gone; now on net IN1_RIGHT: U4.3 (IN1)
- net IN2_A is gone; now on net IN2_RIGHT: U4.2 (IN2)
- net SCL_3V is gone; now on net SCL: U1.23 (SCL)
- net SCL_EXT is gone; now on net GND: U1.7 (AUX_CL)
- net SDA_3V is gone; now on net SDA: U1.24 (SDA)
- net SDA_EXIT is gone; now on net GND: U1.6 (AUX_DA)
- net VCC is gone; now on net +3.3V: C3.1
- net +3.3V: now also A1.2 (3V3), J1.3 (Pin_3), J2.3 (Pin_3), R10.1, R11.1; no longer C5.1
- net GND: now also U1.9 (AD0), C6.2, C7.2, C9.2, H2.1, J1.6 (Pin_6), J2.6 (Pin_6), U2.1 (GND), U2.7 (GND), U2.9 (GND)
- net SCL: now also H3.1, H4.1, R10.2
- net SDA: now also R11.2
- net at U4.6 (OUT1): now also J2.1 (Pin_1)
- net at U4.8 (OUT2): now also J2.2 (Pin_2)
- net OUT_B_LEFT: now reaches A1.10 (IO4/A5)
- net OUT_B_LEFT: now also J1.5 (Pin_5)
- net IN1_RIGHT: now reaches A1.19 (A6/IO14)
- net IN2_RIGHT: now reaches A1.20 (A7/IO32)
- net IN1_LEFT: now reaches A1.21 (A8/IO15)
- net IN1_LEFT: now also U2.3 (IN1)
- net IN2_LEFT: now reaches A1.22 (A9/IO33)
- net IN2_LEFT: now also U2.2 (IN2)
- net OUT_A_RIGHT: now reaches A1.7 (I34/A2)
- net OUT_A_RIGHT: now also J2.4 (Pin_4)
- net OUT_B_RIGHT: now reaches A1.8 (I39/A3)
- net OUT_B_RIGHT: now also J2.5 (Pin_5)
- net OUT_A_LEFT: now reaches A1.9 (IO36/A4)
- net OUT_A_LEFT: now also J1.4 (Pin_4)
- net AD0: no longer names the net of R1.1
- net AD0: now also U2.4 (ILIM); no longer U1.9 (AD0)
- net MOTOR_POWER renamed 12V_BAT
- net 12V_BAT: now also C5.1, C6.1, C7.1, C9.1, U2.5 (VM)
- new net: J1.1 (Pin_1), U2.6 (OUT1)
- new net: J1.2 (Pin_2), U2.8 (OUT2)
- new net +3V3: H1.1
Other:
- note added: "GPIO 13 BATTERY VOLTAGE"
- note added: "IMU BREAKOUT BACKUP"
- note added: "IMU I2C PULLUPS"
- note added: "LEFT MOTOR"
- note added: "MOTOR POWER"
- note added: "RIGHT MOTOR"
- note removed: "2X C7 CLOSE TO EACH DRIVER"
- note removed: "I2C ADDRESS"
- note removed: "I2C PULLUPS & SHIFT"
- note removed: "MOTOR DRIVER"
- note removed: "POWER SUPPLY"
- moved on the sheet: A1, C1, C2, D1, J3, R2, R8, U1, U4

Commit message: board stuff
Parts:
- removed H1, H2, H3, H4: MountingHole_Pad, symbol Mechanical:MountingHole_Pad
- added J4: Conn_01x08_Socket, Connector_PinSocket_1.00mm:PinSocket_1x08_P1.00mm_Vertical, symbol Connector:Conn_01x08_Socket
- C7, C9: footprint (none) -> Capacitor_SMD:CP_Elec_5x5.3
- J1, J2: footprint TerminalBlock_Phoenix:TerminalBlock_Phoenix_PT-1,5-6-3.5-H_1x06_P3.50mm_Horizontal -> TerminalBlock_Phoenix:TerminalBlock_Phoenix_MPT-0,5-6-2.54_1x06_P2.54mm_Horizontal
- J3: footprint (none) -> TerminalBlock_Phoenix:TerminalBlock_Phoenix_MPT-0,5-2-2.54_1x02_P2.54mm_Horizontal
Connections:
- net +3V3: now also J4.1 (Pin_1)
- net GND: now also J4.2 (Pin_2)
- net SCL: now also J4.3 (Pin_3)
- net SDA: now also J4.4 (Pin_4)

Commit message: board design
Connections:
- net +3V3 is gone; now on net +3.3V: J4.1 (Pin_1)
Changed lines of the file:
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@@
+    )
+  )
+  (symbol (lib_id "power:+3.3V") (at 30.48 172.72 90) (unit 1)
+    (in_bom yes) (on_board yes) (dnp no) (fields_autoplaced)
+    (property "Reference" "#PWR012" (at 34.29 172.72 0)
+      (effects (font (size 1.27 1.27)) hide)
+    )
+    (property "Value" "+3.3V" (at 26.67 172.72 90)
+      (effects (font (size 1.27 1.27)) (justify left))
+    )
+    (property "Footprint" "" (at 30.48 172.72 0)
+      (effects (font (size 1.27 1.27)) hide)
+    )
+    (property "Datasheet" "" (at 30.48 172.72 0)
+      (effects (font (size 1.27 1.27)) hide)
+    )
+    (pin "1")
+    (instances
+      (project "Balance_Bot"
+        (path "/983de3f5-cd8b-4631-a29e-093bfdfe9949"
+          (reference "#PWR012") (unit 1)
+        )
+      )
     )
   )
@@
         )
       )
-    )
-  )
-  (symbol (lib_id "power:+3V3") (at 30.48 172.72 90) (unit 1)
-    (in_bom yes) (on_board yes) (dnp no) (fields_autoplaced)
-    (property "Reference" "#PWR020" (at 34.29 172.72 0)
-      (effects (font (size 1.27 1.27)) hide)
-    )
-    (property "Value" "+3V3" (at 26.67 172.72 90)
-      (effects (font (size 1.27 1.27)) (justify left))
-    )
-    (property "Footprint" "" (at 30.48 172.72 0)
-      (effects (font (size 1.27 1.27)) hide)
-    )
-    (property "Datasheet" "" (at 30.48 172.72 0)
-      (effects (font (size 1.27 1.27)) hide)
-    )
-    (pin "1")
-    (instances
-      (project "Balance_Bot"
-        (path "/983de3f5-cd8b-4631-a29e-093bfdfe9949"
-          (reference "#PWR020") (unit 1)
-        )
-      )

Commit message: board
Parts:
- added H1, H2, H3, H4: MountingHole, MountingHole:MountingHole_3.2mm_M3, symbol Mechanical:MountingHole
- C5, C6: value 0.1uF/12V -> 0.1uF/16V
- C7, C9: value 47uF/12V -> 47uF/16V; footprint Capacitor_SMD:CP_Elec_5x5.3 -> Capacitor_THT:CP_Radial_D6.3mm_P2.50mm
- J4: footprint Connector_PinSocket_1.00mm:PinSocket_1x08_P1.00mm_Vertical -> Connector_PinSocket_2.54mm:PinSocket_1x08_P2.54mm_Vertical
Other:
- note added: "DRV8871 SCHEMATIC PER ADAFRUIT"
- note added: "MPU-6050 SCHEMATIC PER ADAFRUIT"
- note removed: "MPU-6050"
Changed lines of the file:
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@@
     (stroke (width 0) (type default))
   )
-  (wire (pts (xy 143.51 153.67) (xy 149.86 153.67))
+  (wire (pts (xy 139.7 153.67) (xy 149.86 153.67))
     (stroke (width 0) (type default))
   )
@@
     (stroke (width 0) (type default))
   )
-  (wire (pts (xy 143.51 160.02) (xy 143.51 153.67))
+  (wire (pts (xy 139.7 160.02) (xy 139.7 153.67))
     (stroke (width 0) (type default))
   )
@@
     (effects (font (size 1.27 1.27)) (justify left bottom))
   )
-  (text "MPU-6050" (at 198.12 83.82 0)
+  (text "MPU-6050\nSCHEMATIC PER ADAFRUIT" (at 184.15 83.82 0)
     (effects (font (size 1.27 1.27)) (justify left bottom))
   )
   (text "MOTOR POWER" (at 228.6 80.01 0)
+    (effects (font (size 1.27 1.27)) (justify left bottom))
+  )
+  (text "DRV8871 \nSCHEMATIC PER ADAFRUIT" (at 146.05 166.37 0)
     (effects (font (size 1.27 1.27)) (justify left bottom))
   )
@@
     )
   )
+  (symbol (lib_id "Mechanical:MountingHole") (at 21.59 129.54 0) (unit 1)
+    (in_bom yes) (on_board yes) (dnp no) (fields_autoplaced)
+    (property "Reference" "H4" (at 24.13 128.27 0)
+      (effects (font (size 1.27 1.27)) (justify left))
+    )
+    (property "Value" "MountingHole" (at 24.13 130.81 0)
+      (effects (font (size 1.27 1.27)) (justify left))
+    )
+    (property "Footprint" "MountingHole:MountingHole_3.2mm_M3" (at 21.59 129.54 0)
+      (effects (font (size 1.27 1.27)) hide)
+    )
+    (property "Datasheet" "~" (at 21.59 129.54 0)
+      (effects (font (size 1.27 1.27)) hide)
+    )
+    (instances
+      (project "Balance_Bot"
+        (path "/983de3f5-cd8b-4631-a29e-093bfdfe9949"
+          (reference "H4") (unit 1)
+        )
+      )
+    )
+  )
   (symbol (lib_id "power:+3.3V") (at 252.73 77.47 0) (unit 1)
     (in_bom yes) (on_board yes) (dnp no)
@@
     )
   )
-  (symbol (lib_id "power:GND") (at 143.51 160.02 0) (unit 1)
-    (in_bom yes) (on_board yes) (dnp no) (fields_autoplaced)
-    (property "Reference" "#PWR023" (at 143.51 166.37 0)
-      (effects (font (size 1.27 1.27)) hide)
-    )
-    (property "Value" "GND" (at 143.51 165.1 0)
-      (effects (font (size 1.27 1.27)))
-    )
-    (property "Footprint" "" (at 143.51 160.02 0)
-      (effects (font (size 1.27 1.27)) hide)
-    )
-    (property "Datasheet" "" (at 143.51 160.02 0)
+  (symbol (lib_id "power:GND") (at 139.7 160.02 0) (unit 1)
+    (in_bom yes) (on_board yes) (dnp no) (fields_autoplaced)
+    (property "Reference" "#PWR023" (at 139.7 166.37 0)
+      (effects (font (size 1.27 1.27)) hide)
+    )
+    (property "Value" "GND" (at 139.7 165.1 0)
+      (effects (font (size 1.27 1.27)))
+    )
+    (property "Footprint" "" (at 139.7 160.02 0)
+      (effects (font (size 1.27 1.27)) hide)
+    )
+    (property "Datasheet" "" (at 139.7 160.02 0)
       (effects (font (size 1.27 1.27)) hide)
     )
@@
       (effects (font (size 1.27 1.27)))
     )
-    (property "Value" "47uF/12V" (at 214.63 125.73 90)
-      (effects (font (size 1.27 1.27)))
-    )
-    (property "Footprint" "Capacitor_SMD:CP_Elec_5x5.3" (at 218.44 129.8448 0)
+    (property "Value" "47uF/16V" (at 214.63 125.73 90)
+      (effects (font (size 1.27 1.27)))
+    )
+    (property "Footprint" "Capacitor_THT:CP_Radial_D6.3mm_P2.50mm" (at 218.44 129.8448 0)
       (effects (font (size 1.27 1.27)) hide)
     )
@@
       (effects (font (size 1.27 1.27)) (justify left))
     )
-    (property "Footprint" "Connector_PinSocket_1.00mm:PinSocket_1x08_P1.00mm_Vertical" (at 40.64 180.34 0)
+    (property "Footprint" "Connector_PinSocket_2.54mm:PinSocket_1x08_P2.54mm_Vertical" (at 40.64 180.34 0)
       (effects (font (size 1.27 1.27)) hide)
     )
@@
       (effects (font (size 1.27 1.27)))
     )
-    (property "Value" "0.1uF/12V" (at 195.58 125.73 90)
+    (property "Value" "0.1uF/16V" (at 195.58 125.73 90)
       (effects (font (size 1.27 1.27)))
     )
@@
       (effects (font (size 1.27 1.27)))
     )
-    (property "Value" "0.1uF/12V" (at 105.41 125.73 90)
+    (property "Value" "0.1uF/16V" (at 105.41 125.73 90)
       (effects (font (size 1.27 1.27)))
     )
@@
     )
   )
+  (symbol (lib_id "Mechanical:MountingHole") (at 21.59 124.46 0) (unit 1)
+    (in_bom yes) (on_board yes) (dnp no) (fields_autoplaced)
+    (property "Reference" "H3" (at 24.13 123.19 0)
+      (effects (font (size 1.27 1.27)) (justify left))
+    )
+    (property "Value" "MountingHole" (at 24.13 125.73 0)
+      (effects (font (size 1.27 1.27)) (justify left))
+    )
+    (property "Footprint" "MountingHole:MountingHole_3.2mm_M3" (at 21.59 124.46 0)
+      (effects (font (size 1.27 1.27)) hide)
+    )
+    (property "Datasheet" "~" (at 21.59 124.46 0)
+      (effects (font (size 1.27 1.27)) hide)
+    )
+    (instances
+      (project "Balance_Bot"
+        (path "/983de3f5-cd8b-4631-a29e-093bfdfe9949"
+          (reference "H3") (unit 1)
+        )
+      )
+    )
+  )
   (symbol (lib_id "power:GND") (at 182.88 43.18 90) (mirror x) (unit 1)
     (in_bom yes) (on_board yes) (dnp no)
@@
         (path "/983de3f5-cd8b-4631-a29e-093bfdfe9949"
           (reference "#PWR019") (unit 1)
+        )
+      )
+    )
+  )
+  (symbol (lib_id "Mechanical:MountingHole") (at 21.59 114.3 0) (unit 1)
+    (in_bom yes) (on_board yes) (dnp no) (fields_autoplaced)
+    (property "Reference" "H1" (at 24.13 113.03 0)
+      (effects (font (size 1.27 1.27)) (justify left))
+    )
+    (property "Value" "MountingHole" (at 24.13 115.57 0)
+      (effects (font (size 1.27 1.27)) (justify left))
+    )
+    (property "Footprint" "MountingHole:MountingHole_3.2mm_M3" (at 21.59 114.3 0)
+      (effects (font (size 1.27 1.27)) hide)
+    )
+    (property "Datasheet" "~" (at 21.59 114.3 0)
+      (effects (font (size 1.27 1.27)) hide)
+    )
+    (instances
+      (project "Balance_Bot"
+        (path "/983de3f5-cd8b-4631-a29e-093bfdfe9949"
+          (reference "H1") (unit 1)
         )
       )
@@
     )
   )
+  (symbol (lib_id "Mechanical:MountingHole") (at 21.59 119.38 0) (unit 1)
+    (in_bom yes) (on_board yes) (dnp no) (fields_autoplaced)
+    (property "Reference" "H2" (at 24.13 118.11 0)
+      (effects (font (size 1.27 1.27)) (justify left))
+    )
+    (property "Value" "MountingHole" (at 24.13 120.65 0)
+      (effects (font (size 1.27 1.27)) (justify left))
+    )
+    (property "Footprint" "MountingHole:MountingHole_3.2mm_M3" (at 21.59 119.38 0)
+      (effects (font (size 1.27 1.27)) hide)
+    )
+    (property "Datasheet" "~" (at 21.59 119.38 0)
+      (effects (font (size 1.27 1.27)) hide)
+    )
+    (instances
+      (project "Balance_Bot"
+        (path "/983de3f5-cd8b-4631-a29e-093bfdfe9949"
+          (reference "H2") (unit 1)
+        )
+      )
+    )
+  )
   (symbol (lib_id "Device:C_Polarized") (at 124.46 130.81 90) (unit 1)
     (in_bom yes) (on_board yes) (dnp no)
@@
       (effects (font (size 1.27 1.27)))
     )
-    (property "Value" "47uF/12V" (at 124.46 125.73 90)
-      (effects (font (size 1.27 1.27)))
-    )
-    (property "Footprint" "Capacitor_SMD:CP_Elec_5x5.3" (at 128.27 129.8448 0)
-      (effects (font (size 1.27 1.27)) hide)
-    )
+    (property "Value" "47uF/16V" (at 124.46 125.73 90)
+      (effects (font (size 1.27 1.27)))
+    )
+    (property "Footprint" "Capacitor_THT:CP_Radial_D6.3mm_P2.50mm" (at 128.27 129.8448 0)
+      (effects (font (size 1.27 1.27)) hide)
+    )

Commit message: Board stuff
Connections:
- net INT: now also A1.23 (A10/IO27), J4.8 (Pin_8)
Other:
- moved on the sheet: C1, C2, C3, C4, J4, U1

Commit message: final board
Parts:
- added H5, H6: IMU MountingHole, MountingHole:MountingHole_3.2mm_M3, symbol Mechanical:MountingHole
Changed lines of the file:
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@@
+    )
+  )
+  (symbol (lib_id "Mechanical:MountingHole") (at 21.59 139.7 0) (unit 1)
+    (in_bom yes) (on_board yes) (dnp no) (fields_autoplaced)
+    (property "Reference" "H6" (at 24.13 138.43 0)
+      (effects (font (size 1.27 1.27)) (justify left))
+    )
+    (property "Value" "IMU MountingHole" (at 24.13 140.97 0)
+      (effects (font (size 1.27 1.27)) (justify left))
+    )
+    (property "Footprint" "MountingHole:MountingHole_3.2mm_M3" (at 21.59 139.7 0)
+      (effects (font (size 1.27 1.27)) hide)
+    )
+    (property "Datasheet" "~" (at 21.59 139.7 0)
+      (effects (font (size 1.27 1.27)) hide)
+    )
+    (instances
+      (project "Balance_Bot"
+        (path "/983de3f5-cd8b-4631-a29e-093bfdfe9949"
+          (reference "H6") (unit 1)
+        )
+      )
     )
   )
@@
         )
       )
+    )
+  )
+  (symbol (lib_id "Mechanical:MountingHole") (at 21.59 134.62 0) (unit 1)
+    (in_bom yes) (on_board yes) (dnp no) (fields_autoplaced)
+    (property "Reference" "H5" (at 24.13 133.35 0)
+      (effects (font (size 1.27 1.27)) (justify left))
+    )
+    (property "Value" "IMU MountingHole" (at 24.13 135.89 0)
+      (effects (font (size 1.27 1.27)) (justify left))
+    )
+    (property "Footprint" "MountingHole:MountingHole_3.2mm_M3" (at 21.59 134.62 0)
+      (effects (font (size 1.27 1.27)) hide)
+    )
+    (property "Datasheet" "~" (at 21.59 134.62 0)
+      (effects (font (size 1.27 1.27)) hide)
+    )
+    (instances
+      (project "Balance_Bot"
+        (path "/983de3f5-cd8b-4631-a29e-093bfdfe9949"
+          (reference "H5") (unit 1)
+        )
+      )
